Commit message: update er12; update codes for ease of use when switching from er7 to er12.

File: er12_description/urdf/er12_support/er12.urdf (robot description, URDF)
Before this commit: robot er12, 9 links, 8 joints
Joints:
- joint joint_1: axis 0 0 1 -> 0 0 -1
- joint joint_2: axis 0 0 1 -> 0 0 -1
- joint joint_3: axis 0 0 1 -> 0 0 -1
- joint joint_4: axis 0 0 1 -> 0 0 -1
- joint joint_5: axis 0 0 1 -> 0 0 -1
- joint joint_6: axis 0 0 1 -> 0 0 -1

File: er12_description/urdf/er12_support/er12.xacro (robot description, xacro)
@@ -86,5 +86,5 @@
 		<joint type="revolute" name="${prefix}joint_1">
 		  <origin xyz="0 0 0" rpy="0 0 0"/>
-		  <axis xyz="0 0 1"/>
+                  <axis xyz="0 0 -1"/>
 		  <parent link="${prefix}base_link"/>
 		  <child link="${prefix}link_1"/>
@@ -93,5 +93,5 @@
 		<joint type="revolute" name="${prefix}joint_2">
 		  <origin xyz="${DH_L6} 0 ${DH_L1}" rpy="${M_PI/2} 0 0"/>
-		  <axis xyz="0 0 1"/>
+                  <axis xyz="0 0 -1"/>
 		  <parent link="${prefix}link_1"/>
 		  <child link="${prefix}link_2"/>
@@ -100,5 +100,5 @@
 		<joint type="revolute" name="${prefix}joint_3">
 		  <origin xyz="0 ${DH_L2} 0" rpy="0 0 ${M_PI/2}"/>
-		  <axis xyz="0 0 1"/>
+                  <axis xyz="0 0 -1"/>
 		  <parent link="${prefix}link_2"/>
 		  <child link="${prefix}link_3"/>
@@ -107,5 +107,5 @@
 		<joint type="revolute" name="${prefix}joint_4">
 		  <origin xyz="${DH_L3} 0 0" rpy="${M_PI/2} 0 0"/>
-		  <axis xyz="0 0 1"/>
+                  <axis xyz="0 0 -1"/>
 		  <parent link="${prefix}link_3"/>
 		  <child link="${prefix}link_4"/>
@@ -114,5 +114,5 @@
 		<joint type="revolute" name="${prefix}joint_5">
 		  <origin xyz="0 0 ${DH_L4}" rpy="-${M_PI/2} 0 0"/>
-		  <axis xyz="0 0 1"/>
+                  <axis xyz="0 0 -1"/>
 		  <parent link="${prefix}link_4"/>
 		  <child link="${prefix}link_5"/>
@@ -121,5 +121,5 @@
 		<joint type="revolute" name="${prefix}joint_6">
 		  <origin xyz="0 -${DH_L5} 0" rpy="${M_PI/2} 0 0"/>
-		  <axis xyz="0 0 1"/>
+                  <axis xyz="0 0 -1"/>
 		  <parent link="${prefix}link_5"/>
 		  <child link="${prefix}link_6"/>
